Commit message: Update urdf and launch files

File: urdf/caster.xacro (robot description, xacro)
@@ -28,5 +28,5 @@
       <axis xyz="0 0 1" />
       <limit effort="0.1" velocity="100"/>
-      <dynamics damping="10.0" friction="0.0"/>
+      <dynamics damping="0.1" friction="0.0"/>
     </joint>
     <transmission name="${prefix}_yaw_trans">
@@ -52,5 +52,5 @@
         <origin xyz="0 0 0" rpy="0 0 0" />
         <geometry>
-          <mesh filename="package://iri_segway_rmp200_description/meshes/caster_wheel.dae" scale="0.0254 0.0254 0.0254"/>
+          <mesh filename="package://iri_segway_rmp200_description/meshes/caster_wheel.dae" scale="1 1 1"/>
         </geometry>
         <material name="grey"/>
@@ -59,5 +59,5 @@
         <origin xyz="0 0 0" rpy="1.57 0 0" />
         <geometry>
-          <cylinder length="0.001" radius="0.0782"/>
+          <cylinder length="0.001" radius="0.083"/>
         </geometry>
       </collision>
@@ -69,5 +69,5 @@
       <axis xyz="0 1 0" />
       <limit effort="1" velocity="100"/>
-      <dynamics damping="10.0" friction="0.0"/>
+      <dynamics damping="0.0" friction="0.0"/>
     </joint>
     <transmission name="${prefix}_caster_wheel_trans">

File: urdf/segway_example.xacro (robot description, xacro)
@@ -4,3 +4,5 @@
   <xacro:include filename="$(find iri_segway_rmp200_description)/urdf/segway_rmp200.xacro" />
   <xacro:segway_rmp200 name="$(arg name)" sim_config="$(find iri_diff_drive_gazebo)/config/segway_rmp200.yaml"/>
+  <xacro:include filename="$(find iri_segway_rmp200_description)/urdf/caster_support_wheels.xacro" />
+  <xacro:caster_support_wheels/>
 </robot>

File: urdf/segway_rmp200.xacro (robot description, xacro)
@@ -6,5 +6,5 @@
   <xacro:include filename="$(find iri_segway_rmp200_description)/urdf/caster.xacro" />
   <xacro:macro name="segway_rmp200" params="name sim_config">
-    <xacro:segway_gazebo name="$(arg name)" sim_config="${sim_config}"/>
+    <xacro:segway_gazebo name="${name}" sim_config="${sim_config}"/>
     <material name="grey">
       <color rgba="0.7 0.7 0.7 1"/>
@@ -31,12 +31,12 @@
         <origin xyz="0 0 -0.08" rpy="0 0 0"/>
         <geometry>
-          <mesh filename="package://iri_segway_rmp200_description/meshes/rmp200.stl" scale="1 1 1"/>
+          <mesh filename="package://iri_segway_rmp200_description/meshes/rmp200_nowheels.stl" scale="1 1 1"/>
         </geometry>
         <material name="grey"/>
       </visual>
       <collision>
-        <origin xyz="0 0 0.18" rpy="0 0 0" />
+        <origin xyz="0 0 0.175" rpy="0 0 0" />
         <geometry>
-          <cylinder length="0.65" radius="0.3"/>
+          <box size="0.3 0.4 0.65"/>
         </geometry>
       </collision>
@@ -65,9 +65,15 @@
           izz="0.001"/>
       </inertial>
+      <collision>
+        <origin xyz="0 0 -0.01" rpy="0 0 0" />
+        <geometry>
+          <cylinder length="0.02" radius="0.31"/>
+        </geometry>
+      </collision>
     </link>
     <joint name="base_link2top_plate" type="fixed">
       <parent link="base_link"/>
       <child link="top_plate"/>
-      <origin rpy="0 0 0" xyz="0 0 0.5"/>
+      <origin rpy="0 0 0" xyz="0 0 0.51"/>
       <axis xyz="0 0 1"/>
     </joint>
@@ -81,43 +87,4 @@
       <origin xyz="0 -0.2725 0.0" rpy="0 0 0" />
     </xacro:segway_wheel>
-    <!-- caster support -->
-    <link name="caster_support">
-      <inertial>
-        <origin xyz="0 0 0" rpy="0 0 0"/>
-        <mass value="1"/>
-        <inertia
-          ixx="0.001" ixy="0.0" ixz="0.0"
-          iyy="0.001" iyz="0.0"
-          izz="0.001"/>
-      </inertial>
-      <visual>
-       <origin xyz="0 0 -0.055" rpy="0 0 0" />
-       <geometry>
-         <box size="0.7 0.25 0.03"/>
-       </geometry>
-       <material name="grey"/>
-      </visual>
-      <collision>
-       <origin xyz="0 0 -0.055" rpy="0 0 0" />
-       <geometry>
-         <box size="0.7 0.25 0.03"/>
-       </geometry>
-       <material name="grey"/>
-      </collision>
-    </link>
-    <joint name="base_link2caster_support" type="fixed">
-      <parent link="base_link"/>
-      <child link="caster_support"/>
-      <origin rpy="0 0 0" xyz="0 0 0.005"/>
-      <axis xyz="0 0 1"/>
-    </joint>
-    <!-- front caster set -->
-    <xacro:segway_caster prefix="front" parent="caster_support">
-      <origin xyz="0.3292 0 -0.07" rpy="0 0 3.14159" />
-    </xacro:segway_caster>
-    <!-- rear caster set -->
-    <xacro:segway_caster prefix="rear" parent="caster_support">
-      <origin xyz="-0.3292 0 -0.07" rpy="0 0 0" />
-    </xacro:segway_caster>
   </xacro:macro>
 </robot>

Commit message: Updated meshes, from stl to dae

File: urdf/caster.xacro (robot description, xacro)
@@ -18,5 +18,4 @@
           <mesh filename="package://iri_segway_rmp200_description/meshes/caster_link.dae" scale="0.0254 0.0254 0.0254"/>
         </geometry>
-        <material name="grey"/>
       </visual>
       <!--no collision-->
@@ -54,5 +53,4 @@
           <mesh filename="package://iri_segway_rmp200_description/meshes/caster_wheel.dae" scale="1 1 1"/>
         </geometry>
-        <material name="grey"/>
       </visual>
       <collision>

File: urdf/caster_support_wheels.xacro (robot description, xacro)
@@ -17,5 +17,7 @@
          <box size="0.7 0.25 0.03"/>
        </geometry>
-       <material name="grey"/>
+       <material name="dark_grey">
+         <color rgba="0.2 0.2 0.2 1"/>
+       </material>
       </visual>
       <collision>
@@ -24,5 +26,4 @@
          <box size="0.7 0.25 0.03"/>
        </geometry>
-       <material name="grey"/>
       </collision>
     </link>

File: urdf/segway_rmp200.xacro (robot description, xacro)
@@ -31,7 +31,6 @@
         <origin xyz="0 0 -0.08" rpy="0 0 0"/>
         <geometry>
-          <mesh filename="package://iri_segway_rmp200_description/meshes/rmp200_nowheels.stl" scale="1 1 1"/>
+          <mesh filename="package://iri_segway_rmp200_description/meshes/rmp200_nowheels.dae" scale="1 1 1"/>
         </geometry>
-        <material name="grey"/>
       </visual>
       <collision>
