Commit message: Moved wheel damping parameter definition. Defined support gazebo material

File: urdf/caster_support_wheels.xacro (robot description, xacro)
@@ -28,4 +28,7 @@
       </collision>
     </link>
+    <gazebo reference="caster_support">
+      <material>Gazebo/FlatBlack</material>
+    </gazebo>
     <joint name="base_link2caster_support" type="fixed">
       <parent link="base_link"/>

File: urdf/wheel.xacro (robot description, xacro)
@@ -10,4 +10,5 @@
       <parent link="${parent}" />
       <child link="${prefix}_wheel_link" />
+      <dynamics damping="0.7" friction="0.2" />
     </joint>
     <link name="${prefix}_wheel_link">
