Commit message: Remove intertia from base_footprint link

File: urdf/include/segway_rmp200.xacro (robot description, xacro)
@@ -11,12 +11,4 @@
     </material>
     <link name="base_footprint">
-      <inertial>
-        <mass value="1" />
-        <origin xyz="0.0 0 0.0" />
-        <inertia
-          ixx="0.001" ixy="0.0" ixz="0.0"
-          iyy="0.001" iyz="0.0"
-          izz="0.001" />
-      </inertial>
     </link>
     <link name="base_link">
